File: GroundStation.kicad_sch (KiCad schematic)
At the start: 0 parts

Commit message: First version
Parts:
- added H2, H3, H4: M3, MountingHole:MountingHole_3mm, symbol Mechanical:MountingHole
Other:
- note added: "MOUNTING"
