File: mcu.kicad_sch (KiCad schematic)
At the start: 11 parts

Commit message: First version
Parts:
- removed J?: UART, symbol Connector_Generic:Conn_01x03
- removed J?: SWDIO, symbol Connector_Generic:Conn_01x03
- added J3: UART/BT, Connector_PinSocket_2.54mm:PinSocket_1x06_P2.54mm_Horizontal, symbol Connector_Generic:Conn_01x06
- added J4: DEBUG, Connector_PinSocket_2.54mm:PinSocket_1x04_P2.54mm_Horizontal, symbol Connector_Generic:Conn_01x04
- C1: renamed from C?; footprint (none) -> Capacitor_SMD:C_0603_1608Metric
- C2: renamed from C?; footprint (none) -> Capacitor_SMD:C_0402_1005Metric
- J1: renamed from J?; footprint (none) -> Connector_PinSocket_2.54mm:PinSocket_1x08_P2.54mm_Vertical
- J2: renamed from J?; footprint (none) -> Connector_PinSocket_2.54mm:PinSocket_1x04_P2.54mm_Vertical
- R1, R2, R3, R4: renamed from R?; footprint (none) -> Resistor_SMD:R_0402_1005Metric
- gave numbers to parts that had none: 1
Connections:
- net VCC is gone; now on net +3V3: J1.1 (Pin_1)
- net +3V3: now also J3.2 (Pin_2)
- net GND: now also J3.3 (Pin_3), J4.1 (Pin_1)
- net RX: now also J3.4 (Pin_4)
- net SWC: now also J4.4 (Pin_4)
- net SWD: now also J4.3 (Pin_3)
- net TX: now also J3.5 (Pin_5)
- net RST: now reaches R1.1, U1.5 (PF2-NRST)
- net RST: now also J4.2 (Pin_2)
- net A0 renamed D_A0
- net CS renamed D_CS
- net LED renamed D_LED
- net LED0: no longer names the net of U1.14 (PB0)
- net LED1: no longer names the net of U1.13 (PA7)
- net LED2 renamed GPIO1
- net RESET renamed D_RST
- net SCK renamed D_SCK
- net SDA renamed D_SDA
- new net EN: J3.1 (Pin_1)
- new net STA: J3.6 (Pin_6)
Other:
- note added: "17x40mm"
