File: pwr.kicad_sch (KiCad schematic)
At the start: 9 parts

Commit message: First version
Parts:
- C20, C22: renamed from C?; footprint (none) -> Capacitor_SMD:C_0603_1608Metric
- C21, C23: renamed from C?; value (none) -> 1uF; footprint (none) -> Capacitor_SMD:C_0603_1608Metric
- J6: renamed from J?; footprint (none) -> Connector_PinHeader_2.54mm:PinHeader_1x02_P2.54mm_Vertical
- R6, R7: renamed from R?; footprint (none) -> LED_SMD:LED_0402_1005Metric
- U4: renamed from U?; value (none) -> LP5907MFX-3.3; footprint (none) -> Package_TO_SOT_SMD:SOT-23-5
- gave numbers to parts that had none: 1
