File: trx.kicad_sch (KiCad schematic)
At the start: 29 parts, among them J1 SMA, U2 AS179-92LF, X1 TCXO 26 MHz

Commit message: First version
Parts:
- removed U1: ~, symbol RF:Si4463
- added J7: RFShield_OnePiece, RF_Shielding:Laird_Technologies_BMI-S-205-F_38.10x25.40mm, symbol Device:RFShield_OnePiece
- added U2: Si4463, Package_DFN_QFN:QFN-20-1EP_4x4mm_P0.5mm_EP2.6x2.6mm_ThermalVias, symbol RF:Si4463
- X1: value TCXO 26 MHz -> TCXO 30 MHz; footprint Crystal:Crystal_SMD_2016-4Pin_2.0x1.6mm -> Crystal:Crystal_SMD_2520-4Pin_2.5x2.0mm
- renumbered C3 to C10, C16 to C11, C6 to C12, C17 to C13, C11 to C14, C12 to C15, C9 to C16, C15 to C17, C7 to C18, C8 to C19, C1 to C3, C2 to C4, C4 to C5, C5 to C6, C10 to C7, C13 to C8, C14 to C9, J1 to J5, L2 to L1, L4 to L2, L5 to L3, L6 to L4, L7 to L5, L1 to L6, L3 to L7, R1 to R5, U2 to U3
Connections:
- net +3V3 is gone; now on net +3.3VA: C7.2, R5.1
- net +3.3VA: now also U2.6 (VDD), U2.8 (VDD)
- net GND: now also J7.1 (Shield), U2.18 (GND), U2.21 (GND)
- net GPIO0: now also U2.9 (GPIO0)
- net GPIO1: now also U2.10 (GPIO1)
- net GPIO2: now also U2.19 (GPIO2)
- net GPIO3: now also U2.20 (GPIO3)
- net RF_CS: now also U2.15 (~{SEL})
- net RF_IRQ: now also U2.11 (~{IRQ})
- net RF_MISO: now also U2.13 (SDO)
- net RF_MOSI: now also U2.14 (SDI)
- net RF_SCK: now also U2.12 (SCLK)
- net RF_SDN: now also U2.1 (SDN)
- net RXn: now also U2.3 (RXn)
- net RXp: now also U2.2 (RXp)
- net TX_UM: now also U2.4 (TX)
- net XOUT: now also U2.17 (XIN)
Other:
- note added: "X1G005421031512"
- note removed: "X1G004691001512"
