File: GroundStation.kicad_pcb (KiCad board)
At the start: 2 copper layers, 58 x 72 mm, 53 parts, among them J1 LCD, J2 SD, J3 UART/BT, J4 DEBUG, J5 SMA, J6 BAT, J7 RFShield_OnePiece, U1 STM32G071GBU, U2 Si4463, U3 AS179-92LF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

Commit message: Added project name
Other:
- board text added: "MADE BY BASEMENT PROJECT WASSUP GROUND STATION V1"
Changed lines of the file:
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@@
     (effects (font (size 1 1) (thickness 0.15)) (justify mirror))
+  )
+  (gr_text "MADE BY BASEMENT\nPROJECT WASSUP\nGROUND STATION\nV1" (at 104 69.4) (layer "B.SilkS")
+    (effects (font (size 2 2) (thickness 0.3)) (justify mirror))
   )
   (gr_text "SWD" (at 129 75) (layer "B.SilkS")
